File: hardware/Nano X ESP.kicad_pcb (KiCad board)
At the start: 2 copper layers, 51 parts, among them J1 Conn_ESP, J2 Conn_Atmega, J3 Conn_ESP, J4 Conn_Atmega, J5 Conn_FT232, J6 CONN_SIM800l, J7 CONN_Power, J8 Conn_I2C, J9 Conn_SPI, Q1 S8050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

Commit message: fixed version 1
Parts:
- removed U6: UFL-MALE, DC-DC converter:UFL-Male
- added AE1: Antenna_Shield, Connector_Coaxial:U.FL_Molex_MCRF_73412-0110_Vertical, F.Cu at (185.2, 114.9)
- added J10: Conn_Output, Connector_PinHeader_2.54mm:PinHeader_1x03_P2.54mm_Vertical, F.Cu at (182.9, 81.9)
- C1, C11, C9, JP1, JP2, JP3, JP4, JP5, JP6, R1, R10, R11, R12, R2, R3, R4, R5, R8, R9: moved to B.Cu
- C10: footprint Capacitor_SMD:CP_Elec_4x5.4 -> Capacitor_SMD:C_0805_2012Metric_Pad1.18x1.45mm_HandSolder; moved to B.Cu
- C4, C6, C7, C8: footprint Capacitor_SMD:CP_Elec_4x5.4 -> Capacitor_SMD:C_0805_2012Metric_Pad1.18x1.45mm_HandSolder
- J1, J3: footprint DC-DC converter:PinHeader_1x08_P2.54mm_Vertical -> Connector_PinHeader_2.54mm:PinHeader_1x06_P2.54mm_Vertical
- J2, J4: footprint DC-DC converter:PinHeader_1x13_P2.54mm_Vertical -> Connector_PinHeader_2.54mm:PinHeader_1x11_P2.54mm_Vertical
- J5: footprint DC-DC converter:PinHeader_1x06_P2.54mm_Vertical -> Connector_PinHeader_2.54mm:PinHeader_1x06_P2.54mm_Vertical
- J6: footprint DC-DC converter:PinHeader_1x02_P2.54mm_Vertical -> Connector_PinHeader_2.54mm:PinHeader_1x02_P2.54mm_Vertical
- J7: value CONN_Power -> CONN_Input; footprint DC-DC converter:PinHeader_1x02_P2.54mm_Vertical -> Connector_PinHeader_2.54mm:PinHeader_1x02_P2.54mm_Vertical
- J8: value Conn_I2C -> Conn_SPI; footprint DC-DC converter:PinHeader_1x02_P2.54mm_Vertical -> Connector_PinHeader_2.54mm:PinHeader_1x06_P2.54mm_Vertical
- J9: value Conn_SPI -> Conn_I2C; footprint DC-DC converter:PinHeader_1x04_P2.54mm_Vertical -> Connector_PinHeader_2.54mm:PinHeader_1x04_P2.54mm_Vertical
- Q1, Q2: footprint Package_TO_SOT_THT:TO-92_Inline -> Package_TO_SOT_SMD:SOT-23; moved to B.Cu
- SW1, SW2: footprint Button_Switch_SMD:SW_SPST_CK_RS282G05A3 -> Button_Switch_SMD:SW_SPST_FSMSM
- Y1: value 16MHz -> 16.000 Mhz; footprint Crystal:Crystal_SMD_0603-2Pin_6.0x3.5mm -> Crystal:Crystal_SMD_HC49-SD
- moved H1 166.1 mm to (185.4, 125.1)
- moved J5 112.9 mm to (182.9, 103.5), turned to 180 degrees
- moved U4 112.4 mm to (170.8, 119.4), turned to 0 degrees
- moved J8 104.3 mm to (154.9, 113.0), turned to 0 degrees
- moved J6 95.4 mm to (176.5, 76.2), turned to 90 degrees
- moved C3 87.3 mm to (139.1, 99.3), turned to 270 degrees
- moved H2 82.9 mm to (105.4, 74.9)
- moved J7 82.7 mm to (169.5, 76.2), turned to 90 degrees
- moved Y1 81.2 mm to (130.6, 98.4), turned to 0 degrees
- moved H4 80.5 mm to (105.4, 125.1)
- moved J4 79.2 mm to (118.7, 123.8)
- moved U5 78.6 mm to (165.1, 97.8)
- moved J2 78.6 mm to (146.1, 123.8)
- moved U2 78.0 mm to (131.4, 108.0)
- moved C7 76.2 mm to (126.4, 116.6), turned to 270 degrees
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Connections:
- J1 pad 1: /RST -> /ADCIN
- J1 pad 2: /ADCIN -> /GPIO16
- J1 pad 3: /GPIO16 -> /D13
- J1 pad 4: /D13 -> /D12
- J1 pad 5: /D12 -> /D11
- J1 pad 6: /D11 -> /CS
- J2 pad 1: /D13 -> /A0
- J2 pad 10: /A7 -> /D1
- J2 pad 11: +5V -> /D2
- J2 pad 2: VCC -> /A1
- J2 pad 3: /A0 -> /A2
- J2 pad 4: /A1 -> /A3
- J2 pad 5: /A2 -> /A4
- J2 pad 6: /A3 -> /A5
- J2 pad 7: /A4 -> /A6
- J2 pad 8: /A5 -> /A7
- J2 pad 9: /A6 -> /D0
- J3 pad 1: /D1 -> /D0
- J3 pad 2: /D0 -> /D1
- J4 pad 1: /D12 -> /D13
- J4 pad 10: /D3 -> /D4
- J4 pad 11: /D2 -> /D3
- J4 pad 2: /D11 -> /D12
- J4 pad 3: /CS -> /D11
- J4 pad 4: /D9 -> /CS
- J4 pad 5: /D8 -> /D9
- J4 pad 6: /D7 -> /D8
- J4 pad 7: /D6 -> /D7
- J4 pad 8: /D5 -> /D6
- J4 pad 9: /D4 -> /D5
- J5 pad 1: /D1 -> /D0
- J5 pad 2: /D0 -> /D1
- J8 pad 1: /A5 -> VCC
- J8 pad 2: /A4 -> GND
- J9 pad 1: /D12 -> VCC
- J9 pad 2: /D11 -> GND
- J9 pad 3: /D13 -> /A5
- J9 pad 4: /CS -> /A4
- U4 pad 13: VCC -> +3V3
Routing:
- net GND: track 206.7 -> 64.5 mm, vias 5 -> 45
- net /DTR: track 8.58 -> 118.5 mm, vias 0 -> 1
- net VCC: track 67.8 -> 168.7 mm, vias 3 -> 6
- net /D12: track 38.5 -> 137.1 mm
- net /D11: track 36.7 -> 131.4 mm
- net /D13: track 49.4 -> 139.0 mm
- net /CS: track 62.8 -> 148.2 mm, vias 5 -> 2
- net +3V3: track 32.6 -> 111.1 mm, vias 2 -> 3
- net /A5: track 20.3 -> 77.2 mm, vias 0 -> 2
- net /A4: track 19.3 -> 73.3 mm, vias 0 -> 1
- net /RTS: track 19.9 -> 73.4 mm, vias 2 -> 1
- net /GPIO0: track 60.6 -> 21.7 mm, vias 3 -> 1
- net /D1: track 61.7 -> 97.0 mm, vias 1 -> 2
- net /D0: track 62.9 -> 96.1 mm, vias 1 -> 3
- net /ADCIN: track 36.3 -> 3.44 mm
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- added copper zone on B.Cu, net GND
- added copper zone on F.Cu, net GND
Other:
- board outline added: 88.9 x 59.1 mm
- board text added: "+3.3V"
- board text added: "+4V"
- board text added: "+5V"
- board text added: "A0"
- board text added: "A1"
- board text added: "A2"
- board text added: "A3"
- board text added: "A4"
- board text added: "A5"
- board text added: "A6"
- board text added: "A7"
- board text added: "ADC"
- board text added: "CS"
- board text added: "D0"
- board text added: "D1"
- board text added: "D10"
- board text added: "D11"
- board text added: "D12"
- board text added: "D13"
- board text added: "D2"
- board text added: "D3"
- board text added: "D4"
- board text added: "D5"
- board text added: "D6"
- board text added: "D7"
- board text added: "D8"
- board text added: "D9"
- board text added: "DTR"
- board text added: "GND"
- board text added: "MISO"
- board text added: "MOSI"
- board text added: "RTS"
- board text added: "RX"
- board text added: "SCK"
- board text added: "SCL"
- board text added: "SDA"
- board text added: "TX"
- board text added: "VCC"
