File: hardware/Nano X ESP.sch (KiCad schematic (older format))
At the start: 51 parts, among them J1 Conn_ESP, J2 Conn_Arduino, J3 Conn_ESP, J4 Conn_Arduino, J5 Conn_FT232, J6 CONN_SIM800l, J7 CONN_Power, J8 Conn_I2C, J9 Conn_SPI, Q1 S8050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

Commit message: fixed version 1
Parts:
- removed J1, J3: Conn_ESP, DC-DC converter:PinHeader_1x08_P2.54mm_Vertical, symbol Connector_Generic:Conn_01x08
- removed J2, J4: Conn_Arduino, DC-DC converter:PinHeader_1x15_P2.54mm_Vertical, symbol Connector_Generic:Conn_01x15
- removed J8: Conn_I2C, DC-DC converter:PinHeader_1x02_P2.54mm_Vertical, symbol Connector_Generic:Conn_01x02
- removed U6: UFL-MALE, DC-DC converter:UFL-Male, symbol Connector~UFL:UFL-MALE
- removed Y1: 16MHz, Crystal:Crystal_SMD_0603-2Pin_6.0x3.5mm, symbol Device:Crystal_Small
- added AE1: Antenna_Shield, Connector_Coaxial:U.FL_Molex_MCRF_73412-0110_Vertical, symbol Device:Antenna_Shield
- added J1, J3: Conn_ESP, Connector_PinHeader_2.54mm:PinHeader_1x06_P2.54mm_Vertical, symbol Connector_Generic:Conn_01x06
- added J10: Conn_Output, Connector_PinHeader_2.54mm:PinHeader_1x03_P2.54mm_Vertical, symbol Connector_Generic:Conn_01x03
- added J2, J4: Conn_Atmega, Connector_PinHeader_2.54mm:PinHeader_1x11_P2.54mm_Vertical, symbol Connector_Generic:Conn_01x11
- added J8: Conn_SPI, Connector_PinHeader_2.54mm:PinHeader_1x06_P2.54mm_Vertical, symbol Connector_Generic:Conn_01x06
- added Y1: 16.000 Mhz, Crystal:Crystal_SMD_HC49-SD, symbol Device:Crystal
- C10, C4, C6, C7, C8: footprint Capacitor_SMD:CP_Elec_4x5.4 -> Capacitor_SMD:C_0805_2012Metric_Pad1.18x1.45mm_HandSolder
- J5: footprint DC-DC converter:PinHeader_1x06_P2.54mm_Vertical -> Connector_PinHeader_2.54mm:PinHeader_1x06_P2.54mm_Vertical
- J6: footprint DC-DC converter:PinHeader_1x02_P2.54mm_Vertical -> Connector_PinHeader_2.54mm:PinHeader_1x02_P2.54mm_Vertical
- J7: value CONN_Power -> CONN_Input; footprint DC-DC converter:PinHeader_1x02_P2.54mm_Vertical -> Connector_PinHeader_2.54mm:PinHeader_1x02_P2.54mm_Vertical
- J9: value Conn_SPI -> Conn_I2C; footprint DC-DC converter:PinHeader_1x04_P2.54mm_Vertical -> Connector_PinHeader_2.54mm:PinHeader_1x04_P2.54mm_Vertical
- Q1, Q2: footprint Package_TO_SOT_THT:TO-92_Inline -> Package_TO_SOT_SMD:SOT-23
- SW1, SW2: footprint Button_Switch_SMD:SW_SPST_CK_RS282G05A3 -> Button_Switch_SMD:SW_SPST_FSMSM
Connections:
- net labels removed: REF, VIN
- wire segments 281 -> 275
Other:
- moved on the sheet: C1, C2, C3, J5, J6, J7, JP1, JP2, JP3, JP4, JP5, JP6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
